File: Kicad/_autosave-25v PSU.sch (KiCad schematic (older format))
At the start: 84 parts, among them J1 Conn_01x10_Female, J2 Conn_02x03_Odd_Even, K1 G5V-1, Q1 TIP3055G, Q2 TIP3055G, Q3 MMBT3904, Q4 MMBT3904, SW1 Rotary_Encoder, SW2 Rotary_Encoder, SW3 SW_Mains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

Commit message: design updates
Parts:
- removed C1, C2: 4700uF, Capacitor_THT:C_Radial_D16.0mm_H25.0mm_P7.50mm, symbol Device:C
- removed C3, C4, C5: 470u, Capacitor_THT:C_Radial_D6.3mm_H7.0mm_P2.50mm, symbol Device:C
- added C? (x2): 22p, symbol Device:C
- added C? (x3): 4700uF, symbol Device:CP1
- added C? (x2): 470uF, symbol Device:CP1
- added C?: 1u, symbol Device:C
- added D?: LED, LED_SMD:LED_0603_1608Metric_Pad1.05x0.95mm_HandSolder, symbol Device:LED
- added Q?: MMBT3904, Package_TO_SOT_SMD:SOT-23, symbol Transistor_BJT:MMBT3904
- added R?: 10k, Resistor_SMD:R_0603_1608Metric_Pad1.05x0.95mm_HandSolder, symbol Device:R
- added R?: 330, Resistor_SMD:R_0603_1608Metric_Pad1.05x0.95mm_HandSolder, symbol Device:R
- added R?: 330, symbol Device:R
- Y1: value 8MHz Crystal -> 20MHz Crystal
Connections:
- net 3.3V: now also R?.1
- net GND: now also R25.1, C?.2, C?.2, C?.2, C?.2, C?.2, C?.2, C?.2, C?.2, Q?.2 (E), R?.1; no longer R25.2
- net Io: now also C?.1, R?.2; no longer U4.5 (OUT)
- net MISO: no longer J1.4 (Pin_4)
- net SS0: now also U8.32 (PD2); no longer U8.14 (PB2)
- net XTAL1: now also C?.1
- net XTAL2: now also C?.1
- net unreg: now also C?.1, C?.1
- net at R2.1, R3.2: now also C?.1
- net at Q2.1 (B), R3.1, R4.1: now also C?.1
- net at D1.2 (A), K1.10, Q1.3 (E)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: now also C?.1
- net CurrentLimit: now reaches Q4.1 (B), U10.7
- net CurrentLimit: now also Q?.1 (B)
- net RS: now reaches U8.12 (PB0)
- net RS: now also J1.4 (Pin_4)
- net at U8.24 (PC1): now also D?.2 (A)
- net at U8.31 (PD1): now also Q?.3 (C), R?.2
- net at D8.1 (K): now also R25.2; no longer R25.1
- new net: R?.1, U4.5 (OUT)
- new net: D?.1 (K), R?.2
- no-connect marks 0 -> 1
Other:
- moved on the sheet: C9, D8, R25, U8
