File: Kicad/25v PSU.kicad_pcb (KiCad board)
At the start: 2 copper layers, 139.7 x 63.5 mm, 86 parts, among them J1 Conn_01x10_Female, J2 Conn_02x03_Odd_Even, K1 G5V-1, Q1 TIP3055G, Q2 TIP3055G, Q3 MMBT3904, Q4 MMBT3904, SW1 Rotary_Encoder, SW2 Rotary_Encoder, SW3 SW_Mains, T1 Transformer_1P_1S, U1 LM358, U10 LM358, U11 REF3020, U12 INA219AxD, U2 LM336, U3 MC78M05_TO252, U4 MAX4080T, U5 LT3080xST, U6 MCP4922, U7 LM334Z, U8 ATmega328P-AU, U9 L78L33_SOT89, Y1 8MHz Crystal

Commit message: V2 design complete
Parts:
- removed the REF** at (38.6, 78.7)
- removed the REF** at (33.0, 65.0)
- added C15: 0.1u, Capacitor_SMD:C_0603_1608Metric_Pad1.05x0.95mm_HandSolder, F.Cu at (241.0, 99.9)
- added C16: 100n, Capacitor_SMD:C_0603_1608Metric_Pad1.05x0.95mm_HandSolder, F.Cu at (212.0, 114.9)
- added C17: 100n, Capacitor_SMD:C_0603_1608Metric_Pad1.05x0.95mm_HandSolder, F.Cu at (222.0, 116.0)
- added D10: D, Diode_SMD:D_SOD-123F, F.Cu at (200.0, 73.0)
- added D9: D_Zener, Diode_SMD:D_MiniMELF_Handsoldering, F.Cu at (264.0, 77.8)
- added J3: Conn_02x03, Connector_PinHeader_2.54mm:PinHeader_2x03_P2.54mm_Vertical, F.Cu at (218.0, 154.0)
- added LOGO: , Logos:LOGO16x16, B.Cu at (276.0, 109.0)
- added LOGO: , Logos:LOGO16x16, F.Cu at (244.0, 148.0)
- added Q5: MMBT3904, Package_TO_SOT_SMD:SOT-23_Handsoldering, F.Cu at (210.0, 100.0)
- added R33: 100k, Resistor_SMD:R_0603_1608Metric_Pad1.05x0.95mm_HandSolder, F.Cu at (216.9, 94.0)
- added R34: 4.7k, Resistor_SMD:R_0603_1608Metric_Pad1.05x0.95mm_HandSolder, F.Cu at (258.0, 136.0)
- added R35: 4.7k, Resistor_SMD:R_0603_1608Metric_Pad1.05x0.95mm_HandSolder, F.Cu at (258.0, 134.0)
- added REF**: KiCad-Logo_8mm_SilkScreen, Symbol:KiCad-Logo_8mm_SilkScreen, B.Cu at (264.0, 137.0)
- added REF**: OSHW-Logo2_9.8x8mm_SilkScreen, Symbol:OSHW-Logo2_9.8x8mm_SilkScreen, B.Cu at (268.0, 129.0)
- C1, C2: value 4700uF -> 0.1u; footprint Capacitor_THT:C_Radial_D16.0mm_H25.0mm_P7.50mm -> Capacitor_SMD:C_0603_1608Metric_Pad1.05x0.95mm_HandSolder
- C10: value 1u -> 100n
- C11: value 2.2u -> 470uF; footprint Capacitor_SMD:C_0603_1608Metric_Pad1.05x0.95mm_HandSolder -> Capacitor_THT:CP_Radial_D8.0mm_P3.50mm
- C13, C6, C7: value 100n -> 4700uF; footprint Capacitor_SMD:C_0603_1608Metric_Pad1.05x0.95mm_HandSolder -> Capacitor_THT:CP_Radial_D16.0mm_P7.50mm
- C14: value 0.1u -> 1u
- C3: value 470u -> 1u; footprint Capacitor_THT:C_Radial_D6.3mm_H7.0mm_P2.50mm -> Capacitor_SMD:C_0603_1608Metric_Pad1.05x0.95mm_HandSolder
- C4, C5: value 470u -> 22p; footprint Capacitor_THT:C_Radial_D6.3mm_H7.0mm_P2.50mm -> Capacitor_SMD:C_0603_1608Metric_Pad1.05x0.95mm_HandSolder
- C8: value 0.1u -> 2.2u
- C9: value 0.1u -> 470uF; footprint Capacitor_SMD:C_0603_1608Metric_Pad1.05x0.95mm_HandSolder -> Capacitor_THT:CP_Radial_D8.0mm_P3.50mm
- D1, D2: value D -> LED; footprint Diode_SMD:D_SOD-123F -> LED_SMD:LED_0603_1608Metric_Pad1.05x0.95mm_HandSolder
- D7: value D_Zener -> D; footprint Diode_SMD:D_MiniMELF_Handsoldering -> Diode_SMD:D_SOD-123F
- D8: value LED -> D; footprint LED_SMD:LED_0603_1608Metric_Pad1.05x0.95mm_HandSolder -> Diode_SMD:D_SOD-123F
- H2: footprint MountingHole:MountingHole_2.5mm_Pad_Via -> MountingHole:MountingHole_2.5mm_Pad
- H3: footprint MountingHole:MountingHole_2.5mm_Pad -> MountingHole:MountingHole_4mm_Pad
- H4: footprint MountingHole:MountingHole_2.5mm_Pad_Via -> MountingHole:MountingHole_4mm_Pad
- J2: value Conn_02x03_Odd_Even -> Barrel_Jack; footprint Connector_PinHeader_2.54mm:PinHeader_2x03_P2.54mm_Vertical -> Connector_BarrelJack:BarrelJack_Horizontal
- Q1, Q2: value TIP3055G -> MMBT3904; footprint Package_TO_SOT_THT:TO-247-3_Vertical -> Package_TO_SOT_SMD:SOT-23_Handsoldering
- Q3, Q4: value MMBT3904 -> TIP3055G; footprint Package_TO_SOT_SMD:SOT-23 -> Package_TO_SOT_THT:TO-247-3_Vertical
- R1: value 10kR -> 330
- R10, R8, R9: value 330 -> 1
- R17: value 1 -> 680
- R18: value 180k -> 3k
- R19: value 180k -> 100
- R2, R3: value 220R -> 330
- R20: value 100R -> 27k
- R21, R23: value 1 -> 220R
- R22: value 1 -> 10k
- R24: value 10k -> 100R
- R25: value 330 -> 10kR
- R26: value 4.7k -> 180k
- R27: value 4.7k -> 10k
- R28: value 680 -> 180k
- R29: value 100 -> 10kR
- R31: value 3k -> 68k
- R32: value 10k -> 330
- R4: value 10kR -> 10k
- R5: value 68k -> 330
- R6: value 100k -> 330
- R7: value 27k -> 1
- U1: value LM358 -> ATmega328P-AU; footprint Package_SO:SOIC-8_3.9x4.9mm_P1.27mm -> Package_QFP:TQFP-32_7x7mm_P0.8mm
- U10: value LM358 -> MC78M05_TO252; footprint Package_SO:SOIC-8_3.9x4.9mm_P1.27mm -> Package_TO_SOT_SMD:TO-252-2
- U11: value REF3020 -> INA219AxD; footprint Package_TO_SOT_SMD:SOT-23 -> Package_SO:SOIC-8_3.9x4.9mm_P1.27mm
- U12: value INA219AxD -> MCP4922; footprint Package_SO:SOIC-8_3.9x4.9mm_P1.27mm -> Package_SO:SOIC-14_3.9x8.7mm_P1.27mm
- U2: value LM336 -> LM358; footprint Package_TO_SOT_THT:TO-92_Inline -> Package_SO:SOIC-8_3.9x4.9mm_P1.27mm
- U3: value MC78M05_TO252 -> LM358; footprint Package_TO_SOT_SMD:TO-252-2 -> Package_SO:SOIC-8_3.9x4.9mm_P1.27mm
- U4: value MAX4080T -> LT3080xST; footprint Package_SO:SOIC-8_3.9x4.9mm_P1.27mm -> Package_TO_SOT_SMD:SOT-223
- U5: value LT3080xST -> LM334Z; footprint Package_TO_SOT_SMD:SOT-223 -> Package_TO_SOT_THT:TO-92_Inline
- U6: value MCP4922 -> L78L33_SOT89; footprint Package_SO:SOIC-14_3.9x8.7mm_P1.27mm -> Package_TO_SOT_SMD:SOT-89-3_Handsoldering
- U7: value LM334Z -> LM336
- U8: value ATmega328P-AU -> REF3020; footprint Package_QFP:TQFP-32_7x7mm_P0.8mm -> Package_TO_SOT_SMD:SOT-23_Handsoldering
- U9: value L78L33_SOT89 -> MAX4080T; footprint Package_TO_SOT_SMD:SOT-89-3 -> Package_SO:SOIC-8_3.9x4.9mm_P1.27mm
- Y1: value 8MHz Crystal -> 20MHz Crystal; footprint Crystal:Crystal_HC52-6mm_Vertical -> Crystal:Crystal_HC52-8mm_Vertical
- moved D2 207.0 mm to (251.9, 146.0)
- moved R10 195.3 mm to (237.0, 80.0), turned to 180 degrees
- moved R9 192.8 mm to (237.0, 82.0), turned to 180 degrees
- moved D1 192.4 mm to (251.9, 143.0), turned to 180 degrees
- moved Q1 190.9 mm to (254.0, 97.0), turned to 270 degrees
- moved R8 190.4 mm to (237.0, 84.0), turned to 180 degrees
- moved R27 185.8 mm to (267.0, 98.0), turned to 90 degrees
- moved C4 185.0 mm to (262.9, 126.0), turned to 180 degrees
- moved D3 184.1 mm to (249.6, 66.0), turned to 0 degrees
- moved J1 183.1 mm to (225.0, 156.0), turned to 180 degrees
- moved R4 183.1 mm to (257.0, 97.0), turned to 90 degrees
- moved U4 180.9 mm to (252.0, 78.0)
- moved R26 180.3 mm to (264.1, 97.0), turned to 0 degrees
- moved U12 178.1 mm to (252.0, 115.0)
- moved C3 177.9 mm to (259.1, 81.0), turned to 0 degrees
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Connections:
- C1 pad 1: unreg -> 3.3V
- C10 pad 1: Net-(C10-Pad1) -> 5V
- C12 pad 1: 5V -> 3.3V
- C13 pad 1: 3.3V -> Net-(C13-Pad1)
- C14 pad 1: 3.3V -> Io
- C2 pad 1: unreg -> Sense-
- C2 pad 2: GND -> Sense+
- C3 pad 1: Net-(C3-Pad1) -> Sense-
- C4 pad 1: Net-(C4-Pad1) -> XTAL1
- C5 pad 1: Net-(C5-Pad1) -> XTAL2
- C6 pad 1: Net-(C6-Pad1) -> unreg
- C7 pad 1: 5V -> unreg
- C8 pad 1: Net-(C10-Pad1) -> Net-(C8-Pad1)
- C8 pad 2: Sense+ -> GND
- C9 pad 1: 3.3V -> Net-(C9-Pad1)
- D1 pad 1: unreg -> Net-(D1-Pad1)
- D1 pad 2: Net-(C5-Pad1) -> Net-(D1-Pad2)
- D2 pad 1: unreg -> Net-(D2-Pad1)
- D3 pad 1: unreg -> Sense-
- D3 pad 2: Net-(D3-Pad2) -> Net-(C8-Pad1)
- D4 pad 1: Net-(D2-Pad2) -> unreg
- D4 pad 2: GND -> Net-(D4-Pad2)
- D5 pad 1: Net-(D3-Pad2) -> unreg
- D5 pad 2: GND -> Net-(D5-Pad2)
- D6 pad 1: Net-(C10-Pad1) -> Net-(D4-Pad2)
- D6 pad 2: Net-(C11-Pad1) -> GND
- D7 pad 1: Net-(C11-Pad1) -> Net-(D5-Pad2)
- D8 pad 1: Net-(D8-Pad1) -> unreg
- D8 pad 2: Net-(D8-Pad2) -> GND
- H3 pad 1: Net-(C11-Pad1) -> Net-(C8-Pad1)
- J1 pad 4: MISO -> RS
- J2 pad 1: MISO -> unreg
- J2 pad 2: 3.3V -> GND
- J2 pad 3: SCK -> (no net)
- K1 pad 10: Net-(C5-Pad1) -> Net-(C13-Pad1)
- Q1 pad 1: unreg -> CurrentLimit
- Q1 pad 2: unreg -> GND
- Q1 pad 3: Net-(C5-Pad1) -> Net-(Q1-Pad3)
- Q2 pad 1: Net-(C4-Pad1) -> CurrentLimit
- Q2 pad 2: unreg -> GND
- Q2 pad 3: unreg -> Net-(Q2-Pad3)
- Q3 pad 1: Net-(Q3-Pad1) -> Net-(C11-Pad1)
- Q3 pad 2: Net-(C6-Pad1) -> unreg
- Q3 pad 3: Net-(C5-Pad1) -> Net-(Q3-Pad3)
- Q4 pad 1: Net-(Q4-Pad1) -> Net-(Q3-Pad3)
- Q4 pad 2: GND -> unreg
- Q4 pad 3: Net-(Q4-Pad3) -> Net-(C13-Pad1)
- R1 pad 1: unreg -> Net-(J1-Pad8)
- R1 pad 2: Net-(R1-Pad2) -> 5V
- R10 pad 1: Net-(J1-Pad10) -> Sense-
- R10 pad 2: 5V -> Sense+
- R11 pad 1: Net-(C10-Pad1) -> Sense-
- R12 pad 1: Net-(C10-Pad1) -> Sense-
- R13 pad 1: Net-(C10-Pad1) -> Sense-
- R14 pad 1: Net-(C10-Pad1) -> Sense-
- R15 pad 1: Net-(C10-Pad1) -> Sense-
- R16 pad 1: Net-(C10-Pad1) -> Sense-
- R17 pad 1: Net-(C10-Pad1) -> Net-(Q2-Pad3)
- R17 pad 2: Sense+ -> Net-(R17-Pad2)
- R18 pad 1: Net-(C11-Pad1) -> GND
- R18 pad 2: Voutput -> Net-(R18-Pad2)
- R19 pad 1: Net-(C11-Pad1) -> VSet
- R19 pad 2: Voutput -> Net-(Q2-Pad3)
- R2 pad 1: Net-(C3-Pad1) -> Net-(J1-Pad9)
- R2 pad 2: unreg -> 5V
- R20 pad 1: Net-(R20-Pad1) -> VSet
- R20 pad 2: GND -> Net-(R18-Pad2)
- R21 pad 1: Net-(C10-Pad1) -> Net-(C9-Pad1)
- R21 pad 2: Sense+ -> unreg
- R22 pad 1: Net-(C10-Pad1) -> 3.3V
- R22 pad 2: Sense+ -> RESET
- R23 pad 1: Net-(C10-Pad1) -> Net-(C11-Pad1)
- R23 pad 2: Sense+ -> Net-(C9-Pad1)
- R24 pad 1: Voutput -> Net-(R24-Pad1)
- R25 pad 1: Net-(D8-Pad1) -> Net-(C11-Pad1)
- R26 pad 1: 3.3V -> Net-(C8-Pad1)
- R26 pad 2: SDA0 -> Voutput
- R27 pad 1: 3.3V -> Voutput
- R27 pad 2: SCL0 -> GND
- R28 pad 1: Net-(Q4-Pad3) -> Net-(C8-Pad1)
- R28 pad 2: Net-(R28-Pad2) -> Voutput
- R29 pad 1: VSet -> unreg
- R29 pad 2: Net-(Q4-Pad3) -> Net-(R29-Pad2)
- R3 pad 1: Net-(C4-Pad1) -> Net-(J1-Pad10)
- R3 pad 2: Net-(C3-Pad1) -> 5V
- R30 pad 1: VSet -> Net-(R30-Pad1)
- R30 pad 2: Net-(R30-Pad2) -> GND
- R31 pad 1: GND -> Net-(R31-Pad1)
- R31 pad 2: Net-(R30-Pad2) -> Net-(R30-Pad1)
- R32 pad 1: 3.3V -> Net-(R32-Pad1)
- R32 pad 2: RESET -> Io
- R4 pad 1: Net-(C4-Pad1) -> 3.3V
- R4 pad 2: GND -> Net-(Q1-Pad3)
- R5 pad 1: Net-(R5-Pad1) -> GND
- R5 pad 2: Net-(R5-Pad2) -> Net-(D1-Pad1)
- R6 pad 1: Net-(R6-Pad1) -> GND
- R6 pad 2: Net-(R5-Pad1) -> Net-(D2-Pad1)
- R7 pad 1: Net-(R5-Pad2) -> Sense-
- R7 pad 2: GND -> Sense+
- R8 pad 1: Net-(J1-Pad8) -> Sense-
- R8 pad 2: 5V -> Sense+
- R9 pad 1: Net-(J1-Pad9) -> Sense-
- R9 pad 2: 5V -> Sense+
- T1 pad 3: Net-(D3-Pad2) -> Net-(D5-Pad2)
- T1 pad 4: Net-(D2-Pad2) -> Net-(D4-Pad2)
- U1 pad 1: Net-(R6-Pad1) -> Encoder2B
- U1 pad 2: Net-(R5-Pad2) -> Encoder2A
- U1 pad 3: Net-(R1-Pad2) -> GND
- U1 pad 4: GND -> 3.3V
- U1 pad 5: Net-(C5-Pad1) -> GND
- U1 pad 6: Net-(R6-Pad1) -> 3.3V
- U1 pad 7: Net-(Q3-Pad1) -> XTAL1
- U1 pad 8: unreg -> XTAL2
- U10 pad 1: Net-(R28-Pad2) -> Net-(C16-Pad1)
- U10 pad 2: Net-(R30-Pad2) -> GND
- U10 pad 3: VoRef -> 5V
- U11 pad 1: 3.3V -> GND
- U11 pad 2: 2.048V -> GND
- U11 pad 3: GND -> SDA0
- U12 pad 1: GND -> 3.3V
- U12 pad 2: GND -> Net-(U12-Pad2)
- U12 pad 3: SDA0 -> SS1
- U12 pad 4: SCL0 -> SCK
- U12 pad 5: 3.3V -> MOSI
- U12 pad 6: GND -> Net-(U12-Pad6)
- U12 pad 7: Sense- -> Net-(U12-Pad7)
- U12 pad 8: Sense+ -> GND
- U2 pad 1: (no net) -> Net-(R17-Pad2)
- U2 pad 2: Net-(R1-Pad2) -> Net-(R18-Pad2)
- U2 pad 3: GND -> VoRef
- U3 pad 1: Net-(C6-Pad1) -> Net-(R33-Pad1)
- U3 pad 2: GND -> Net-(R30-Pad1)
- U3 pad 3: 5V -> Net-(R29-Pad2)
- U4 pad 1: Sense+ -> VSet
- U4 pad 2: Sense+ -> Net-(C8-Pad1)
- U4 pad 3: Net-(U4-Pad3) -> Sense-
- U4 pad 4: GND -> Net-(C8-Pad1)
- U5 pad 1: VSet -> Net-(C8-Pad1)
- U5 pad 2: Net-(C11-Pad1) -> Net-(R24-Pad1)
- U5 pad 3: Net-(C10-Pad1) -> GND
- U6 pad 2: Net-(U6-Pad2) -> GND
- U6 pad 3: SS1 -> 5V
- U7 pad 1: Net-(C11-Pad1) -> (no net)
- U7 pad 2: Net-(R20-Pad1) -> Net-(R29-Pad2)
- U8 pad 1: Encoder2B -> 3.3V
- U8 pad 2: Encoder2A -> 2.048V
- U9 pad 1: 3.3V -> Sense+
- U9 pad 2: GND -> Sense+
- U9 pad 3: 5V -> Net-(U9-Pad3)
Routing:
- net Net-(C5-Pad1): track 159.6 -> 0.00 mm, vias 4 -> 0
- net 5V: track 187.2 -> 71.8 mm, vias 3 -> 1
- net GND: track 451.5 -> 557.1 mm, vias 17 -> 102
- net Net-(C13-Pad1): track 0.00 -> 102.2 mm, vias 0 -> 2
- net Io: track 118.4 -> 18.5 mm, vias 7 -> 2
- net Net-(C8-Pad1): track 0.00 -> 72.5 mm, vias 0 -> 13
- net Sense-: track 11.2 -> 68.0 mm
- net 3.3V: track 149.4 -> 200.1 mm, vias 2 -> 8
- net Encoder1A: track 66.7 -> 18.6 mm, vias 1 -> 0
- net Net-(D8-Pad2): track 46.9 -> 0.00 mm, vias 2 -> 0
- net SS0: track 90.3 -> 44.1 mm, vias 4 -> 2
- net Net-(C4-Pad1): track 45.4 -> 0.00 mm
- net Net-(Q1-Pad3): track 0.00 -> 42.2 mm, vias 0 -> 2
- net Net-(R1-Pad2): track 41.8 -> 0.00 mm
- net Net-(C10-Pad1): track 41.8 -> 0.00 mm
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- added copper zone on B.Cu, net Net-(C8-Pad1)
- added copper zone on F.Cu, net Net-(C8-Pad1)
Other:
- board size 139.7 x 63.5 mm -> 100 x 100 mm
- board text added: "Analog"
- board text added: "By Hamish Sams @ hamish.science"
- board text added: "Designed and made by Hamish Sams © 2020"
- board text added: "Designed as open source hardware"
- board text added: "Digital"
- board text added: "Find out more information at https://hamish.science/"
- board text added: "Hammie217/OpenSourcePSU"
- board text added: "Power"
- board text added: "Schematic and PCB designed using KiCad"
- board text added: "Schematic, board and software available on GitHub"
- board text added: "V2.0"
- board text removed: "0-18V 0-1A"
- board text removed: "Blue"
- board text removed: "Brown"
- board text removed: "Designed by Hamish Sams @ Hamish.Science"
- board text removed: "Negative"
- board text removed: "Positive"
- board text removed: "V1.0"
