File: Kicad/25v PSU.sch (KiCad schematic (older format))
At the start: 84 parts, among them J1 Conn_01x10_Female, J2 Conn_02x03_Odd_Even, K1 G5V-1, Q1 TIP3055G, Q2 TIP3055G, Q3 MMBT3904, Q4 MMBT3904, SW1 Rotary_Encoder, SW2 Rotary_Encoder, SW3 SW_Mains, T1 Transformer_1P_1S, U1 LM358, U10 LM358, U11 REF3020, U12 INA219AxD, U2 LM336, U3 MC78M05_TO252, U4 MAX4080T, U5 LT3080xST, U6 MCP4922, U7 LM334Z, U8 ATmega328P-AU, U9 L78L33_SOT89, Y1 8MHz Crystal

Commit message: design updates
Parts:
- U8: symbol MCU_Microchip_ATmega:ATmega328P-AU -> 25v-PSU-rescue:ATmega328P-AU-MCU_Microchip_ATmega
Connections:
- net Sense-: now also C10.1, C8.1, D6.1 (K), R11.1, R12.1, R13.1, R14.1, R15.1, R16.1, R17.1, R21.1, R22.1, R23.1, U5.3 (IN)
- net unreg: no longer Q1.1 (B), Q2.3 (E)
- new net: Q1.1 (B), Q2.3 (E)
Changed lines of the file:
@@
 EESchema Schematic File Version 4
-LIBS:25v PSU-cache
 EELAYER 30 0
 EELAYER END
@@
 Wire Wire Line
 	5700 1400 4900 1400
-Connection ~ 5700 1700
 Wire Wire Line
 	5700 1400 5700 1700
 Wire Wire Line
 	5950 1400 5700 1400
-Connection ~ 6100 1700
 Wire Wire Line
 	6150 1700 6100 1700
@@
 	1    0    0    -1
 $EndComp
-Wire Wire Line
-	5700 1700 6100 1700
 $Comp
 L Transistor_BJT:TIP3055G Q1
@@
 Text GLabel 2950 3800 3    50   Output ~ 0
 Sense+
-Text GLabel 3450 3850 3    50   Output ~ 0
+Text GLabel 3450 3800 3    50   Output ~ 0
 Sense-
 Text GLabel 9850 5700 0    50   Input ~ 0
@@
 SS0
 $Comp
-L MCU_Microchip_ATmega:ATmega328P-AU U8
+L 25v-PSU-rescue:ATmega328P-AU-MCU_Microchip_ATmega U8
 U 1 1 5F71BC6F
 P 1450 5400

Commit message: V2 design complete
Parts:
- removed C1, C2: 4700uF, Capacitor_THT:C_Radial_D16.0mm_H25.0mm_P7.50mm, symbol Device:C
- removed C3: 470u, Capacitor_THT:C_Radial_D6.3mm_H7.0mm_P2.50mm, symbol Device:C
- added C11, C9: 470uF, Capacitor_THT:CP_Radial_D8.0mm_P3.50mm, symbol Device:CP1
- added C13, C6, C7: 4700uF, Capacitor_THT:CP_Radial_D16.0mm_P7.50mm, symbol Device:CP1
- added C14: 1u, Capacitor_SMD:C_0603_1608Metric_Pad1.05x0.95mm_HandSolder, symbol Device:C
- added D2: LED, LED_SMD:LED_0603_1608Metric_Pad1.05x0.95mm_HandSolder, symbol Device:LED
- added D8: D, Diode_SMD:D_SOD-123F, symbol Device:D
- added J2: Barrel_Jack, Connector_BarrelJack:BarrelJack_Horizontal, symbol Connector:Barrel_Jack
- added Q1: MMBT3904, Package_TO_SOT_SMD:SOT-23_Handsoldering, symbol Transistor_BJT:MMBT3904
- added R32, R6: 330, Resistor_SMD:R_0603_1608Metric_Pad1.05x0.95mm_HandSolder, symbol Device:R
- added R4: 10k, Resistor_SMD:R_0603_1608Metric_Pad1.05x0.95mm_HandSolder, symbol Device:R
- C4, C5: value 470u -> 22p; footprint Capacitor_THT:C_Radial_D6.3mm_H7.0mm_P2.50mm -> Capacitor_SMD:C_0603_1608Metric_Pad1.05x0.95mm_HandSolder
- H2: footprint MountingHole:MountingHole_2.5mm_Pad_Via -> MountingHole:MountingHole_2.5mm_Pad
- H3: footprint MountingHole:MountingHole_2.5mm_Pad -> MountingHole:MountingHole_4mm_Pad
- H4: footprint MountingHole:MountingHole_2.5mm_Pad_Via -> MountingHole:MountingHole_4mm_Pad
- Q2: renamed from Q4; footprint Package_TO_SOT_SMD:SOT-23 -> Package_TO_SOT_SMD:SOT-23_Handsoldering
- Q5: renamed from Q3; footprint Package_TO_SOT_SMD:SOT-23 -> Package_TO_SOT_SMD:SOT-23_Handsoldering
- U6: renamed from U9; footprint Package_TO_SOT_SMD:SOT-89-3 -> Package_TO_SOT_SMD:SOT-89-3_Handsoldering
- U8: renamed from U11; footprint Package_TO_SOT_SMD:SOT-23 -> Package_TO_SOT_SMD:SOT-23_Handsoldering
- Y1: value 8MHz Crystal -> 20MHz Crystal; footprint Crystal:Crystal_HC52-6mm_Vertical -> Crystal:Crystal_HC52-8mm_Vertical
- renumbered C9 to C1, C12 to C10, C13 to C12, C14 to C15, C6 to C16, C7 to C17, C8 to C2, C10 to C3, C11 to C8, D8 to D1, D1 to D10, D6 to D3, D2 to D4, D3 to D5, D4 to D6, D5 to D7, D7 to D9, J2 to J3, Q2 to Q3, Q1 to Q4, R8 to R1, R14 to R10, R15 to R11, R16 to R12, R17 to R13, R21 to R14, R22 to R15, R23 to R16, R28 to R17, R31 to R18, R29 to R19, R9 to R2, R30 to R20, R2 to R21, R32 to R22, R3 to R23, R20 to R24, R4 to R25, R18 to R26, R24 to R27, R19 to R28, R1 to R29, R10 to R3, R7 to R30, R5 to R31, R6 to R33, R26 to R34, R27 to R35, R25 to R5, R11 to R7, R12 to R8, R13 to R9, U8 to U1, U3 to U10, U12 to U11, U6 to U12, U10 to U2, U1 to U3, U5 to U4, U7 to U5, U2 to U7, U4 to U9
Connections:
- net 3.3V: now also R4.1
- net Encoder1A: now also U1.26 (PC3); no longer U1.10 (PD6)
- net Encoder1B: now also U1.25 (PC2); no longer U1.9 (PD5)
- net GND: now also R5.1, C11.2, C13.2, C14.2, C6.2, C7.2, C9.2, D8.2 (A), J2.2, Q1.2 (E), R6.1; no longer R5.2
- net Io: now also C14.1, R32.2; no longer U9.5 (OUT)
- net MISO: no longer J1.4 (Pin_4)
- net SS0: now also U1.32 (PD2); no longer U1.14 (PB2)
- net XTAL1: now also C4.1
- net XTAL2: now also C5.1
- net unreg: now also C6.1, C7.1, D8.1 (K), J2.1
- net at R21.1, R23.2: now also C9.1
- net at Q3.1 (B), R23.1, R25.1: now also C11.1; no longer C4.1
- net at D10.2 (A), K1.10, Q4.3 (E)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: now also C13.1; no longer C5.1
- net CurrentLimit: now reaches Q2.1 (B), U2.7
- net CurrentLimit: now also Q1.1 (B)
- net RS: now reaches U1.12 (PB0)
- net RS: now also J1.4 (Pin_4)
- net at U1.24 (PC1): now also D2.2 (A)
- net at U1.31 (PD1): now also Q1.3 (C), R4.2
- net at D1.1 (K): now also R5.2; no longer R5.1
- new net: R32.1, U9.5 (OUT)
- new net: D2.1 (K), R6.2
- no-connect marks 0 -> 1
Other:
- note added: "07/06/2020"
- note added: "2\n"
- note removed: "1"
- note removed: "10/04/2020"
- moved on the sheet: C1, D1, R5, U1, U3C
